File: PCB/hwboard-bike-computer.kicad_pcb (KiCad board)
At the start: 2 copper layers, 277 x 190 mm, 1 part, among them M1 CM0

Commit message: add sensors
Parts:
- removed M1: CM0, hwboard-bike-computer:CM0
- added U1: TESEO-LIV3R, hwboard-bike-computer:TESEOLIV3R, F.Cu at (128.1, 126.2)
- added U2: TPS61089, Package_DFN_QFN:Texas_VQFN-RNR0011A-11, F.Cu at (147.4, 121.3)
- added U3: BQ25622ERYKR, hwboard-bike-computer:BQ25622ERYKR, F.Cu at (140.0, 122.3)
- added U4: MAX17048G+, Package_DFN_QFN:TDFN-8-1EP_2x2mm_P0.5mm_EP0.8x1.2mm, F.Cu at (138.9, 127.2)
- added U5: RASPBERRY_PI_ZERO_2_W, hwboard-bike-computer:MODULE_RASPBERRY_PI_ZERO_2_W, F.Cu at (156.5, 101.0)
